Commit message: Modified cf2x.urdf, velocityAviary and DSLPIDControl for monocopter model.

File: gym_pybullet_drones/assets/cf2x.urdf (robot description, URDF)
Before this commit: robot cf2, 6 links, 5 joints
Links:
- link base_link: geometry collision cylinder length=.025 radius=.06; visual mesh filename=./monocopter.dae scale=1 1 1
